File: kicad/programming.kicad_sch (KiCad schematic)
At the start: 30 parts, among them J1 USB_C_Receptacle, U1 FT2232HQ, U3 93CxxC, U6 LFE5U-85F-6BG381x, U7 W25Q128JVS, X1 ECS-2520MV-120-BL-TR

Commit message: Removed the nDet from the SD-card and added the 12 MHz oscillator as clock input to be fully compatible with the GECKO4 clock inputs
Connections:
- net CLK_12MHz: now reaches U1.2 (OSCI), X1.3 (OUT)
Changed lines of the file:
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@@
   (junction (at 128.27 44.45) (diameter 0) (color 0 0 0 0)
+  )
+  (junction (at 97.79 165.1) (diameter 0) (color 0 0 0 0)
   )
   (junction (at 90.17 120.65) (diameter 0) (color 0 0 0 0)
@@
     (stroke (width 0) (type default))
   )
+  (wire (pts (xy 101.6 172.72) (xy 97.79 172.72))
+    (stroke (width 0) (type default))
+  )
   (wire (pts (xy 93.98 24.13) (xy 100.33 24.13))
     (stroke (width 0) (type default))
@@
     (stroke (width 0) (type default))
   )
+  (wire (pts (xy 97.79 172.72) (xy 97.79 165.1))
+    (stroke (width 0) (type default))
+  )
   (wire (pts (xy 73.66 107.95) (xy 81.28 107.95))
     (stroke (width 0) (type default))
@@
     (stroke (width 0) (type default))
   )
+  (global_label "CLK_12MHz" (shape output) (at 101.6 172.72 0) (fields_autoplaced)
+    (effects (font (size 1.27 1.27)) (justify left))
+    (property "Intersheetrefs" "${INTERSHEET_REFS}" (at 115.2705 172.72 0)
+      (effects (font (size 1.27 1.27)) (justify left) hide)
+    )
+  )
   (global_label "FTDI_TDO" (shape input) (at 173.99 59.69 0) (fields_autoplaced)
