File: kicad/GECKO5Education/pmod.kicad_sch (KiCad schematic)
At the start: 24 parts, among them J3 Conn_02x06_Odd_Even, J4 Conn_02x06_Odd_Even, J6 Conn_01x08_Socket, U13 NCP1529A, U14 NCP1529A, U6 LFE5U-85F-6BG381x, U8 LP5907MFX-2.5, X1 ECS-2520MV-500-BL-TR

Commit message: Made an alternative version
Parts:
- removed SD1: 104031-0811, gecko4education:microsd, symbol gecko5education:micro_sd
- added SW6: B3U-1000P[], gecko5:SW_B3U-100P_OMR, symbol cpuAddOn:B3U-1000P[]
Connections:
- net GND: now also SW6.2
- net at U6.M5 (PL77A): now also SW6.1
- net SD_CLK renamed red1
- net SD_CMD renamed red2
- net SD_D0 renamed red0
- net SD_D1 renamed green4
- net SD_D2: no longer names the net of U6.J5 (PL50B)
- net SD_D3 renamed red3
- no-connect marks 4 -> 1
Other:
- moved on the sheet: U6A
