File: kicad/GECKO5Education/pmod.kicad_sch (KiCad schematic)
At the start: 31 parts, among them J4 Conn_02x09_Odd_Even, SW6 B3U-1000P[], U13 NCP1529A, U14 NCP1529A, U18 MCP7940MT-I/SN, U6 LFE5U-85F-6BG381x, U8 LP5907MFX-2.5, X2 ECS-2520MV-500-BL-TR, X3 CB3LV-3I-74M2500, X4 ECS-2520MV-240-BL-TR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

Commit message: latest version with camera
Parts:
- removed U18: MCP7940MT-I/SN, gecko4education:SOIC8-N_MC_MCH, symbol gecko5education:MCP7940MT-I_SN
- added BT1: Battery_Cell, Battery:BatteryHolder_Keystone_2998_1x6.8mm, symbol Device:Battery_Cell
- added U18: DS1338Z-33+T&R, gecko4education:DS1338Z-33&plus_T&R, symbol addOnTemplate:DS1338Z-33+T&R
Connections:
- net +3.3V: now also U18.8 (VCC)
- net GND: now also BT1.2 (-), U18.4 (GND)
- net RTC_MFP: now also U18.7 (SQW/OUT)
- net SCL: now also U18.6 (SCL)
- net SDA: now also U18.5 (SDA)
- net at C33.1, Y1.1: now also U18.2 (X2)
- net at C34.1, Y1.2: now also U18.1 (X1)
- new net: BT1.1 (+), U18.3 (VBAT)
- no-connect marks 5 -> 4
Changed lines of the file:
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@@
   (junction (at 205.74 127) (diameter 0) (color 0 0 0 0)
+  )
+  (junction (at 62.23 189.23) (diameter 0) (color 0 0 0 0)
   )
   (junction (at 52.07 189.23) (diameter 0) (color 0 0 0 0)
@@
   (no_connect (at 243.84 91.44))
   (no_connect (at 205.74 34.29))
-  (no_connect (at 69.85 180.34))
   (no_connect (at 48.26 35.56))
   (no_connect (at 54.61 73.66))
@@
     (stroke (width 0) (type default))
   )
-  (wire (pts (xy 52.07 175.26) (xy 69.85 175.26))
+  (wire (pts (xy 52.07 175.26) (xy 80.01 175.26))
     (stroke (width 0) (type default))
   )
@@
     (stroke (width 0) (type default))
   )
+  (wire (pts (xy 80.01 189.23) (xy 80.01 182.88))
+    (stroke (width 0) (type default))
+  )
   (wire (pts (xy 49.53 151.13) (xy 49.53 153.67))
     (stroke (width 0) (type default))
@@
     (stroke (width 0) (type default))
   )
-  (wire (pts (xy 69.85 182.88) (xy 69.85 189.23))
-    (stroke (width 0) (type default))
-  )
   (wire (pts (xy 120.65 102.87) (xy 120.65 104.14))
     (stroke (width 0) (type default))
@@
     (stroke (width 0) (type default))
   )
+  (wire (pts (xy 62.23 180.34) (xy 62.23 181.61))
+    (stroke (width 0) (type default))
+  )
   (wire (pts (xy 241.3 83.82) (xy 243.84 83.82))
     (stroke (width 0) (type default))
@@
     (stroke (width 0) (type default))
   )
+  (wire (pts (xy 62.23 189.23) (xy 80.01 189.23))
+    (stroke (width 0) (type default))
+  )
   (wire (pts (xy 240.03 60.96) (xy 243.84 60.96))
     (stroke (width 0) (type default))
@@
     (stroke (width 0) (type default))
   )
+  (wire (pts (xy 80.01 180.34) (xy 62.23 180.34))
+    (stroke (width 0) (type default))
+  )
   (wire (pts (xy 113.03 19.05) (xy 113.03 20.32))
     (stroke (width 0) (type default))
@@
     (stroke (width 0) (type default))
   )
-  (wire (pts (xy 69.85 189.23) (xy 58.42 189.23))
+  (wire (pts (xy 58.42 189.23) (xy 62.23 189.23))
     (stroke (width 0) (type default))
   )
@@
     (stroke (width 0) (type default))
   )
-  (wire (pts (xy 69.85 177.8) (xy 49.53 177.8))
+  (wire (pts (xy 49.53 177.8) (xy 80.01 177.8))
     (stroke (width 0) (type default))
   )
@@
     )
   )
-  (symbol (lib_id "gecko5education:MCP7940MT-I_SN") (at 69.85 175.26 0) (unit 1)
-    (in_bom yes) (on_board yes) (dnp no) (fields_autoplaced)
-    (property "Reference" "U18" (at 97.79 165.1 0)
-      (effects (font (size 1.524 1.524)))
-    )
-    (property "Value" "MCP7940MT-I/SN" (at 97.79 167.64 0)
-      (effects (font (size 1.524 1.524)))
-    )
-    (property "Footprint" "gecko4education:SOIC8-N_MC_MCH" (at 69.85 175.26 0)
-      (effects (font (size 1.27 1.27) italic) hide)
-    )
-    (property "Datasheet" "MCP7940MT-I/SN" (at 69.85 175.26 0)
-      (effects (font (size 1.27 1.27) italic) hide)
-    )
-    (pin "3")
-    (pin "5")
-    (pin "2")
-    (pin "4")
-    (pin "8")
-    (pin "1")
-    (pin "7")
-    (pin "6")
-    (instances
-      (project "gecko5education"
-        (path "/47d58937-9286-45a8-b88f-d3fcc6f916c8/e8cfb843-efab-422d-aa9c-640a59ac0396"
-          (reference "U18") (unit 1)
-        )
-      )
-    )
-  )
   (symbol (lib_id "Regulator_Switching:NCP1529A") (at 66.04 140.97 0) (unit 1)
     (in_bom yes) (on_board yes) (dnp no) (fields_autoplaced)
@@
         (path "/47d58937-9286-45a8-b88f-d3fcc6f916c8/e8cfb843-efab-422d-aa9c-640a59ac0396"
           (reference "U14") (unit 1)
+        )
+      )
+    )
+  )
+  (symbol (lib_id "addOnTemplate:DS1338Z-33+T&R") (at 80.01 175.26 0) (unit 1)
+    (in_bom yes) (on_board yes) (dnp no) (fields_autoplaced)
+    (property "Reference" "U18" (at 102.87 165.1 0)
+      (effects (font (size 1.524 1.524)))
+    )
+    (property "Value" "DS1338Z-33+T&R" (at 102.87 167.64 0)
+      (effects (font (size 1.524 1.524)))
+    )
+    (property "Footprint" "gecko4education:DS1338Z-33&plus_T&R" (at 102.87 169.164 0)
+      (effects (font (size 1.524 1.524)) hide)
+    )
+    (property "Datasheet" "" (at 80.01 175.26 0)
+      (effects (font (size 1.524 1.524)))
+    )
+    (pin "8")
+    (pin "1")
+    (pin "5")
+    (pin "6")
+    (pin "7")
+    (pin "4")
+    (pin "3")
+    (pin "2")
+    (instances
+      (project "gecko5education"
+        (path "/47d58937-9286-45a8-b88f-d3fcc6f916c8/e8cfb843-efab-422d-aa9c-640a59ac0396"
+          (reference "U18") (unit 1)
         )
       )
@@
         )
       )
+    )
+  )
+  (symbol (lib_id "Device:Battery_Cell") (at 62.23 186.69 0) (unit 1)
+    (in_bom yes) (on_board yes) (dnp no) (fields_autoplaced)
+    (property "Reference" "BT1" (at 66.04 183.5785 0)
+      (effects (font (size 1.27 1.27)) (justify left))
+    )
+    (property "Value" "Battery_Cell" (at 66.04 186.1185 0)
+      (effects (font (size 1.27 1.27)) (justify left))
+    )
+    (property "Footprint" "Battery:BatteryHolder_Keystone_2998_1x6.8mm" (at 62.23 185.166 90)
+      (effects (font (size 1.27 1.27)) hide)
+    )
+    (property "Datasheet" "~" (at 62.23 185.166 90)
+      (effects (font (size 1.27 1.27)) hide)
+    )
+    (pin "1")
+    (pin "2")
+    (instances
+      (project "gecko5education"
+        (path "/47d58937-9286-45a8-b88f-d3fcc6f916c8/e8cfb843-efab-422d-aa9c-640a59ac0396"
+          (reference "BT1") (unit 1)
+        )
+      )
