File: kicad/GECKO5Education/programming.kicad_sch (KiCad schematic)
At the start: 33 parts, among them J1 USB_C_Receptacle, U1 FT2232HQ, U15 FSUSB30UMX, U3 93CxxC, U6 LFE5U-85F-6BG381x, U7 W25Q128JVS, X1 ECS-2520MV-120-BL-TR

Commit message: Made an alternative version
Connections:
- no-connect marks 35 -> 36
Changed lines of the file:
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@@
   (no_connect (at 171.45 135.89))
   (no_connect (at 171.45 128.27))
+  (no_connect (at 50.8 165.1))
   (no_connect (at 45.72 73.66))
   (no_connect (at 171.45 69.85))
