File: kicad/GECKO5Education/programming.kicad_sch (KiCad schematic)
At the start: 33 parts, among them J1 USB_C_Receptacle, U1 FT2232HQ, U15 FSUSB30UMX, U3 93CxxC, U6 LFE5U-85F-6BG381x, U7 W25Q128JVS, X1 ECS-2520MV-120-BL-TR

Commit message: Made version V1.5
Connections:
- net HDMI_nReset: now reaches R1.1, U6.Y3 (DONE)
Changed lines of the file:
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@@
   (junction (at 232.41 104.14) (diameter 0) (color 0 0 0 0)
+  )
+  (junction (at 203.2 41.91) (diameter 0) (color 0 0 0 0)
   )
   (junction (at 223.52 52.07) (diameter 0) (color 0 0 0 0)
@@
     (stroke (width 0) (type default))
   )
+  (wire (pts (xy 195.58 41.91) (xy 203.2 41.91))
+    (stroke (width 0) (type default))
+  )
   (wire (pts (xy 146.05 44.45) (xy 148.59 44.45))
     (stroke (width 0) (type default))
@@
       (effects (font (size 1.27 1.27)) (justify right) hide)
     )
+  )
+  (global_label "HDMI_nReset" (shape output) (at 195.58 41.91 180) (fields_autoplaced)
+    (effects (font (size 1.27 1.27)) (justify right))
+    (property "Intersheetrefs" "${INTERSHEET_REFS}" (at 180.6205 41.91 0)
+      (effects (font (size 1.27 1.27)) (justify right) hide)
+    )

Commit message: Final version
Parts:
- renumbered C1 to C10, C1 to C11, C1 to C12, C1 to C13, C1 to C14, C1 to C9, D122 to D123, R2 to R1, R1 to R116, R1 to R117, R4 to R15, R1 to R18, R1 to R19, R3 to R2, R1 to R20, R1 to R21, R1 to R22, R1 to R23, R1 to R24, R1 to R25, R1 to R26, R1 to R27, R1 to R3, R1 to R5, R1 to R6, U3 to U1, U1 to U2

Commit message: Merged perif-add-on to GECKO5
Parts:
- removed D123: SBA0530Q_R1_00001, Diode_SMD:D_0402_1005Metric, symbol Device:D
- removed R15: 10k, Resistor_SMD:R_0402_1005Metric, symbol Device:R
- removed U15: FSUSB30UMX, gecko4education:IC_FSUSB30UMX, symbol gecko5education:FSUSB30UMX
Connections:
- net +5V: now also J1.A4 (VBUS), J1.A9 (VBUS), J1.B4 (VBUS), J1.B9 (VBUS)
- net UsbD+: now also U2.8 (DP)
- net UsbD-: now also U2.7 (DM)
- net D1+: now reaches J1.A6 (D+), J1.B6 (D+)
- net D1-: now reaches J1.A7 (D-), J1.B7 (D-)

Commit message: Changed the USB-reset to reset the FPGA to reconfigure instead of applying the "reset" button, which makes more sense in a system reset
Connections:
- net nProgramFpga: now reaches R18.1, U6.W3 (~{PROGRAM})
Changed lines of the file:
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@@
   (junction (at 172.72 113.03) (diameter 0) (color 0 0 0 0)
+  )
+  (junction (at 198.12 36.83) (diameter 0) (color 0 0 0 0)
   )
   (junction (at 146.05 44.45) (diameter 0) (color 0 0 0 0)
@@
     (stroke (width 0) (type default))
   )
+  (wire (pts (xy 194.31 36.83) (xy 198.12 36.83))
+    (stroke (width 0) (type default))
+  )
   (wire (pts (xy 133.35 161.29) (xy 135.89 161.29))
     (stroke (width 0) (type default))
@@
       (effects (font (size 1.27 1.27)) (justify right) hide)
     )
+  )
+  (global_label "nProgramFpga" (shape input) (at 194.31 36.83 180) (fields_autoplaced)
+    (effects (font (size 1.27 1.27)) (justify right))
+    (property "Intersheetrefs" "${INTERSHEET_REFS}" (at 177.6575 36.83 0)
+      (effects (font (size 1.27 1.27)) (justify right) hide)
+    )
