File: kicad/GECKO5Education/hdmi.kicad_sch (KiCad schematic)
At the start: 20 parts, among them J2 HDMI_A, U3 PCA9306DQER, U6 LFE5U-85F-6BG381x

Commit message: Made version V1.5
Parts:
- removed C1, C2, C3, C4, C5, C6, C7, C8: 22n, Capacitor_SMD:C_0402_1005Metric, symbol Device:C
- removed D1: BZT52C3V6LP-7, Diode_SMD:D_0402_1005Metric, symbol Device:D_Zener
- removed R10, R11, R8, R9: 4k7, Resistor_SMD:R_0402_1005Metric, symbol Device:R
- removed R12, R14: 549, Resistor_SMD:R_0402_1005Metric, symbol Device:R
- removed R13: 10k, Resistor_SMD:R_0402_1005Metric, symbol Device:R
- removed R7: 100k, Resistor_SMD:R_0402_1005Metric, symbol Device:R
- removed U3: PCA9306DQER, Package_SON:X2SON-8_1.4x1mm_P0.35mm, symbol Interface:PCA9306
- added R1 (x3): 4k7, Resistor_SMD:R_0402_1005Metric, symbol Device:R
- added R1: 10k, Resistor_SMD:R_0402_1005Metric, symbol Device:R
- added R1: 4k3, Resistor_SMD:R_0402_1005Metric, symbol Device:R
- added R1 (x2): 2k2, Resistor_SMD:R_0402_1005Metric, symbol Device:R
- added U3: SII9022ACNU, gecko4education:QFN72_10X10_LAT-M, symbol gecko5education:SII9022ACNU
Connections:
- net +3.3V: now also R1.2, R1.2, U3.21 (IOVCC), U3.3 (IOVCC), U3.46 (IOVCC)
- net +5V: now also R1.2, R1.2
- net GND: now also R1.1, R1.1, R1.1, U3.10 (D18), U3.11 (D17), U3.13 (D16), U3.20 (D9), U3.23 (D8), U3.30 (D2), U3.31 (D1), U3.32 (D0), U3.36 (SPDIF), U3.37 (SD3), U3.39 (SD2), U3.40 (SD1), U3.43 (CGND), U3.57 (IOGND), U3.63 (AGND), U3.69 (IO_SEL), U3.70 (VDDQ), U3.73 (GND)
- net at J2.13 (CEC): now also U3.71 (CEC_A)
- net CK+: now reaches J2.10 (CK+)
- net CK+: now also U3.59 (TXC+)
- net CK-: now reaches J2.12 (CK-)
- net CK-: now also U3.58 (TXC-)
- net TX2+: now reaches J2.1 (D2+)
- net TX2+: now also U3.68 (TX2+)
- net TX1-: now reaches J2.6 (D1-)
- net TX1-: now also U3.64 (TX1-)
- net TX0+: now reaches J2.7 (D0+)
- net TX0+: now also U3.62 (TX0+)
- net TX1+: now reaches J2.4 (D1+)
- net TX1+: now also U3.65 (TX1+)
- net at J2.15 (SCL): now also R1.1, U3.49 (DSCL)
- net at J2.16 (SDA): now also R1.1, U3.48 (DSDA)
- net at J2.19 (HPD): now also R1.2, U3.54 (HPD)
- net TX2-: now reaches J2.3 (D2-)
- net TX2-: now also U3.67 (TX2-)
- net TX0-: now reaches J2.9 (D0-)
- net TX0-: now also U3.61 (TX0-)
- net hdmi_cec renamed HDMI_Blue0
- net HDMI_Blue0: now also U3.29 (D3)
- net hdmi_clk+ renamed HDMI_De
- net HDMI_De: now also U3.33 (DE)
- net hdmi_clk- renamed HDMI_Blue1
- net HDMI_Blue1: now also U3.28 (D4)
- net hdmi_d0+ renamed HDMI_Vsync
- net HDMI_Vsync: now also U3.35 (VSYNC)
- net hdmi_d0- renamed HDMI_Hsync
- net HDMI_Hsync: now also U3.34 (HSYNC)
- net hdmi_d1+ renamed HDMI_Sd0
- net HDMI_Sd0: now also U3.41 (SD0)
- net hdmi_d1- renamed HDMI_Mclk
- net HDMI_Mclk: now also U3.38 (MCLK)
- net hdmi_d2+ renamed HDMI_Sck
- net HDMI_Sck: now also U3.45 (SCK)
- net hdmi_d2- renamed HDMI_Ws
- net HDMI_Ws: now also U3.44 (WS)
- net hdmi_hpd renamed HDMI_Clk
- net HDMI_Clk: now also U3.22 (IDCK)
- net hdmi_scl renamed HDMI_CEC
- net HDMI_CEC: now also U3.50 (CEC_D)
- net hdmi_sda renamed HDMI_Blue3
- net HDMI_Blue3: now also U3.25 (D6)
- net hdmi_util renamed HDMI_Blue2
- net HDMI_Blue2: now also U3.27 (D5)
- new net: R1.2, U3.56 (EXT_SWING)
- new net: R1.2, U3.72 (CI2CA)
- new net +1V2: U3.12 (CVCC12), U3.26 (CVCC12), U3.42 (CVCC12), U3.47 (CVCC12), U3.5 (CVCC12), U3.53 (CVCC12), U3.60 (AVCC12), U3.66 (AVCC12)
- new net HDMI_Blue4: U3.24 (D7)
- new net HDMI_Green0: U3.19 (D10)
- new net HDMI_Green1: U3.18 (D11)
- new net HDMI_Green2: U3.17 (D12)
- new net HDMI_Green3: U3.16 (D13)
- new net HDMI_Green4: U3.15 (D14)
- new net HDMI_Green5: U3.14 (D15)
- new net HDMI_Red0: U3.9 (D19)
- new net HDMI_Red1: U3.8 (D20)
- new net HDMI_Red2: U3.7 (D21)
- new net HDMI_Red3: U3.6 (D22)
- new net HDMI_Red4: U3.4 (D23)
- new net HDMI_SCL: R1.1, U3.1 (CSCL)
- new net HDMI_SDA: R1.1, U3.2 (CSDA)
- new net HDMI_nReset: U3.51 (RESET#)
- no-connect marks 1 -> 3
Other:
- moved on the sheet: J2, U6C

Commit message: Made V1.6
Parts:
- removed R1 (x3): 4k7, Resistor_SMD:R_0402_1005Metric, symbol Device:R
- removed R1: 10k, Resistor_SMD:R_0402_1005Metric, symbol Device:R
- removed R1: 4k3, Resistor_SMD:R_0402_1005Metric, symbol Device:R
- removed R1 (x2): 2k2, Resistor_SMD:R_0402_1005Metric, symbol Device:R
- removed U3: SII9022ACNU, gecko4education:QFN72_10X10_LAT-M, symbol gecko5education:SII9022ACNU
- added C1, C2, C4, C5, C6: 100n, Capacitor_SMD:C_0402_1005Metric, symbol Device:C
- added C29, C3, C7, C8: 100n, Resistor_SMD:R_0402_1005Metric, symbol Device:C
- added J6: Conn_01x06_Socket, Connector_PinSocket_2.54mm:PinSocket_1x06_P2.54mm_Horizontal, symbol Connector:Conn_01x06_Socket
- added R4 (x6): 10k, Resistor_SMD:R_0402_1005Metric, symbol Device:R
- added R4: 33k, Resistor_SMD:R_0402_1005Metric, symbol Device:R
- added R4: 510E, Resistor_SMD:R_0402_1005Metric, symbol Device:R
- added U16: LTC2632CTS8-LZ12TRMPBF, gecko4education:SOT65P280X100-8N, symbol gecko5education:LTC2632CTS8-LZ12TRMPBF
- added U17: MAX11666AUBV, gecko4education:SOP50P490X110-11N, symbol gecko5education:MAX11666AUBV
- added U3: SII164CTG64, gecko4education:QFP50P1200X1200X120-64N, symbol gecko5education:SII164CTG64
Connections:
- net +3.3V: now also C1.2, C2.2, C29.2, C3.2, C4.2, C5.2, C6.2, C7.2, R4.1, R4.2, R4.2, R4.2, R4.2, R4.2, U16.7 (VCC), U17.5 (VDD), U17.8 (OVDD), U3.1 (VCC), U3.12 (VCC), U3.18 (PVCC1), U3.23 (AVCC), U3.29 (AVCC), U3.33 (VCC), U3.49 (PVCC2)
- net GND: now also C1.1, C2.1, C29.1, C3.1, C4.1, C5.1, C6.1, C7.1, C8.1, J6.4 (Pin_4), R4.2, R4.2, U16.4 (GND), U17.11 (EPAD), U17.3 (AGND), U3.16 (GND), U3.17 (PGND), U3.20 (AGND), U3.26 (AGND), U3.32 (AGND), U3.34 (RESERVED), U3.41 (D18), U3.42 (D17), U3.43 (D16), U3.48 (GND), U3.52 (D9), U3.53 (D8), U3.56 (IDCK-), U3.6 (CTL3/A3/DK3), U3.61 (D2), U3.62 (D1), U3.63 (D0), U3.64 (GND), U3.7 (CTL2/A2/DK2), U3.8 (CTL1/A1/DK1)
- net HDMI_Blue0: now also U3.60 (D3); no longer U6.A18 (PT119A)
- net HDMI_Blue1: now also U3.59 (D4); no longer U6.B18 (PT116B)
- net HDMI_Blue2: now also U3.58 (D5); no longer U6.A19 (PT121A)
- net HDMI_Blue3: now also U3.55 (D6); no longer U6.B19 (PT119B)
- net HDMI_Blue4: now also U3.54 (D7)
- net HDMI_Clk: now also U3.57 (IDCK+); no longer U6.B20 (PT121B)
- net HDMI_De: now also U3.2 (DE); no longer U6.A17 (PT116A)
- net HDMI_Green0: now also U3.51 (D10)
- net HDMI_Green1: now also U3.50 (D11)
- net HDMI_Green2: now also U3.47 (D12)
- net HDMI_Green3: now also U3.46 (D13)
- net HDMI_Green4: now also U3.45 (D14)
- net HDMI_Green5: now also U6.B20 (PT121B), U3.44 (D15)
- net HDMI_Hsync: now also U3.4 (HSYNC); no longer U6.B16 (PT110B)
- net HDMI_Red0: now also U6.B19 (PT119B), U3.40 (D19)
- net HDMI_Red1: now also U6.A19 (PT121A), U3.39 (D20)
- net HDMI_Red2: now also U6.B18 (PT116B), U3.38 (D21)
- net HDMI_Red3: now also U6.A18 (PT119A), U3.37 (D22)
- net HDMI_Red4: now also U6.A17 (PT116A), U3.36 (D23)
- net HDMI_Vsync: now also U3.5 (VSYNC); no longer U6.A16 (PT110A)
- net TX0+: now also U3.25 (TX0+)
- net TX0-: now also U3.24 (TX0-)
- net TX1+: now also U3.28 (TX1+)
- net TX1-: now also U3.27 (TX1-)
- net TX2+: now also U3.31 (TX2+)
- net TX2-: now also U3.30 (TX2-)
- net CK+ renamed TXC+
- net TXC+: now also U3.22 (TXC+)
- net CK- renamed TXC-
- net TXC-: now also U3.21 (TXC-)
- net HDMI_CEC renamed ADC_nCS
- net ADC_nCS: now also U17.6 (~{CS})
- net HDMI_Mclk renamed DAC_SCK
- net DAC_SCK: now also U16.1 (SCK)
- net HDMI_Sck renamed ADC_CHSEL
- net ADC_CHSEL: now also U17.7 (CHSEL)
- net HDMI_Sd0 renamed ADC_SDO
- net ADC_SDO: now also U17.9 (DOUT)
- net HDMI_Ws renamed ADC_SCK
- net ADC_SCK: now also U17.10 (SCLK)
- new net: R4.2, U3.10 (~{PD})
- new net: R4.1, U3.13 (ISEL/~{RST})
- new net: R4.1, U3.14 (DSEL/SDA)
- new net: R4.1, U3.15 (BSEL/SCL)
- new net: R4.1, U3.19 (EXT_SWING)
- new net: R4.1, U3.3 (VREF)
- new net: R4.1, U3.35 (DKEN)
- new net: R4.1, U3.9 (EDGE/HTPLG)
- new net ADC_ChanA: J6.2 (Pin_2), U17.1 (AIN1)
- new net ADC_ChanB: J6.3 (Pin_3), U17.2 (AIN2)
- new net DAC_ChanA: J6.5 (Pin_5), U16.5 (VOUTA)
- new net DAC_ChanB: J6.6 (Pin_6), U16.6 (VOUTB)
- new net DAC_SDI: U16.8 (SDI), U6.A16 (PT110A)
- new net DAC_nCS: U16.2 (~CS/LD), U6.B16 (PT110B)
- new net VREF: C8.2, J6.1 (Pin_1), U16.3 (REF), U17.4 (REF)
- no-connect marks 3 -> 2
Other:
- moved on the sheet: U6C

Commit message: No changes
Parts:
- added J7: Conn_01x02_Pin, Connector_PinHeader_1.27mm:PinHeader_1x02_P1.27mm_Horizontal, symbol Connector:Conn_01x02_Pin
Connections:
- net +3.3V: no longer R4.2
- net GND: now also R4.2
- net VREF: now also J7.1 (Pin_1)
- new net +2V5: J7.2 (Pin_2)
Changed lines of the file:
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@@
   (junction (at 256.54 19.05) (diameter 0) (color 0 0 0 0)
   )
-  (junction (at 232.41 118.11) (diameter 0) (color 0 0 0 0)
-  )
   (junction (at 106.68 88.9) (diameter 0) (color 0 0 0 0)
   )
@@
   )
   (junction (at 160.02 52.07) (diameter 0) (color 0 0 0 0)
+  )
+  (junction (at 231.14 120.65) (diameter 0) (color 0 0 0 0)
   )
   (junction (at 208.28 130.81) (diameter 0) (color 0 0 0 0)
@@
     (stroke (width 0) (type default))
   )
-  (wire (pts (xy 231.14 125.73) (xy 231.14 115.57))
+  (wire (pts (xy 231.14 125.73) (xy 231.14 120.65))
     (stroke (width 0) (type default))
   )
@@
     (stroke (width 0) (type default))
   )
-  (wire (pts (xy 232.41 120.65) (xy 226.06 120.65))
-    (stroke (width 0) (type default))
-  )
   (wire (pts (xy 33.02 57.15) (xy 35.56 57.15))
     (stroke (width 0) (type default))
@@
     (stroke (width 0) (type default))
   )
+  (wire (pts (xy 129.54 152.4) (xy 129.54 154.94))
+    (stroke (width 0) (type default))
+  )
   (wire (pts (xy 207.01 46.99) (xy 210.82 46.99))
     (stroke (width 0) (type default))
@@
     (stroke (width 0) (type default))
   )
+  (wire (pts (xy 129.54 157.48) (xy 129.54 171.45))
+    (stroke (width 0) (type default))
+  )
   (wire (pts (xy 160.02 49.53) (xy 161.29 49.53))
     (stroke (width 0) (type default))
@@
     (stroke (width 0) (type default))
   )
-  (wire (pts (xy 232.41 118.11) (xy 232.41 120.65))
-    (stroke (width 0) (type default))
-  )
   (wire (pts (xy 78.74 33.02) (xy 76.2 33.02))
     (stroke (width 0) (type default))
@@
     (stroke (width 0) (type default))
   )
+  (wire (pts (xy 231.14 120.65) (xy 231.14 115.57))
+    (stroke (width 0) (type default))
+  )
   (wire (pts (xy 33.02 72.39) (xy 35.56 72.39))
     (stroke (width 0) (type default))
@@
   )
   (wire (pts (xy 33.02 105.41) (xy 35.56 105.41))
+    (stroke (width 0) (type default))
+  )
+  (wire (pts (xy 226.06 120.65) (xy 231.14 120.65))
     (stroke (width 0) (type default))
   )
@@
     )
   )
+  (symbol (lib_id "Connector:Conn_01x02_Pin") (at 134.62 157.48 180) (unit 1)
+    (in_bom yes) (on_board yes) (dnp no)
+    (property "Reference" "J7" (at 138.43 163.83 0)
+      (effects (font (size 1.27 1.27)))
+    )
+    (property "Value" "Conn_01x02_Pin" (at 140.97 161.29 0)
+      (effects (font (size 1.27 1.27)))
+    )
+    (property "Footprint" "Connector_PinHeader_1.27mm:PinHeader_1x02_P1.27mm_Horizontal" (at 134.62 157.48 0)
+      (effects (font (size 1.27 1.27)) hide)
+    )
+    (property "Datasheet" "~" (at 134.62 157.48 0)
+      (effects (font (size 1.27 1.27)) hide)
+    )
+    (pin "1")
+    (pin "2")
+    (instances
+      (project "gecko5education"
+        (path "/47d58937-9286-45a8-b88f-d3fcc6f916c8/e24858e6-e459-4033-a46a-6eb11205cf28"
+          (reference "J7") (unit 1)
+        )
+      )
+    )
+  )
   (symbol (lib_id "Device:C") (at 250.19 25.4 180) (unit 1)
     (in_bom yes) (on_board yes) (dnp no)
@@
         )
       )
+    )
+  )
+  (symbol (lib_id "power:+2V5") (at 129.54 152.4 0) (unit 1)
+    (in_bom yes) (on_board yes) (dnp no) (fields_autoplaced)
+    (property "Reference" "#PWR038" (at 129.54 156.21 0)
+      (effects (font (size 1.27 1.27)) hide)
+    )
+    (property "Value" "+2V5" (at 129.54 148.59 0)
+      (effects (font (size 1.27 1.27)))
+    )
+    (property "Footprint" "" (at 129.54 152.4 0)
+      (effects (font (size 1.27 1.27)) hide)
+    )
+    (property "Datasheet" "" (at 129.54 152.4 0)
+      (effects (font (size 1.27 1.27)) hide)
+    )
+    (pin "1")
+    (instances
+      (project "gecko5education"
+        (path "/47d58937-9286-45a8-b88f-d3fcc6f916c8/e8cfb843-efab-422d-aa9c-640a59ac0396"
+          (reference "#PWR038") (unit 1)
+        )
+        (path "/47d58937-9286-45a8-b88f-d3fcc6f916c8/e24858e6-e459-4033-a46a-6eb11205cf28"
+          (reference "#PWR0101") (unit 1)
+        )
+      )
