File: kicad/GECKO5Education/gpio.kicad_sch (KiCad schematic)
At the start: 4 parts, among them J5 QSE-020-01-XXX-D, U6 LFE5U-85F-6BG381x

Commit message: small update on V1.4
Parts:
- added D125: SBA0530Q_R1_00001, Diode_SMD:D_0402_1005Metric, symbol Device:D
Connections:
- net +5V: now also D125.2 (A)
- net at D124.2 (A), J5.34: no longer J5.32
- new net: D125.1 (K), J5.32
Other:
- moved on the sheet: D124
Changed lines of the file:
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@@
   (junction (at 97.79 130.81) (diameter 0) (color 0 0 0 0)
   )
-  (junction (at 95.25 109.22) (diameter 0) (color 0 0 0 0)
-  )
   (junction (at 97.79 128.27) (diameter 0) (color 0 0 0 0)
   )
+  (junction (at 125.73 107.95) (diameter 0) (color 0 0 0 0)
+  )
   (junction (at 214.63 50.8) (diameter 0) (color 0 0 0 0)
   )
@@
     (stroke (width 0) (type default))
   )
-  (wire (pts (xy 95.25 109.22) (xy 95.25 110.49))
-    (stroke (width 0) (type default))
-  )
   (wire (pts (xy 200.66 148.59) (xy 204.47 148.59))
     (stroke (width 0) (type default))
@@
     (stroke (width 0) (type default))
   )
-  (wire (pts (xy 95.25 107.95) (xy 95.25 109.22))
-    (stroke (width 0) (type default))
-  )
   (wire (pts (xy 95.25 105.41) (xy 97.79 105.41))
     (stroke (width 0) (type default))
@@
     (stroke (width 0) (type default))
   )
+  (wire (pts (xy 124.46 110.49) (xy 125.73 110.49))
+    (stroke (width 0) (type default))
+  )
   (wire (pts (xy 200.66 146.05) (xy 204.47 146.05))
     (stroke (width 0) (type default))
   )
+  (wire (pts (xy 116.84 106.68) (xy 113.03 106.68))
+    (stroke (width 0) (type default))
+  )
   (wire (pts (xy 95.25 97.79) (xy 97.79 97.79))
     (stroke (width 0) (type default))
@@
     (stroke (width 0) (type default))
   )
-  (wire (pts (xy 116.84 109.22) (xy 95.25 109.22))
-    (stroke (width 0) (type default))
-  )
   (wire (pts (xy 200.66 115.57) (xy 204.47 115.57))
     (stroke (width 0) (type default))
@@
     (stroke (width 0) (type default))
   )
+  (wire (pts (xy 113.03 106.68) (xy 113.03 107.95))
+    (stroke (width 0) (type default))
+  )
   (wire (pts (xy 200.66 140.97) (xy 204.47 140.97))
     (stroke (width 0) (type default))
@@
     (stroke (width 0) (type default))
   )
+  (wire (pts (xy 95.25 107.95) (xy 113.03 107.95))
+    (stroke (width 0) (type default))
+  )
   (wire (pts (xy 109.22 69.85) (xy 95.25 69.85))
     (stroke (width 0) (type default))
@@
     (stroke (width 0) (type default))
   )
+  (wire (pts (xy 124.46 106.68) (xy 125.73 106.68))
+    (stroke (width 0) (type default))
+  )
   (wire (pts (xy 25.4 118.11) (xy 25.4 50.8))
     (stroke (width 0) (type default))
@@
     (stroke (width 0) (type default))
   )
+  (wire (pts (xy 125.73 107.95) (xy 125.73 110.49))
+    (stroke (width 0) (type default))
+  )
   (wire (pts (xy 97.79 128.27) (xy 97.79 130.81))
     (stroke (width 0) (type default))
@@
     (stroke (width 0) (type default))
   )
+  (wire (pts (xy 125.73 106.68) (xy 125.73 107.95))
+    (stroke (width 0) (type default))
+  )
   (wire (pts (xy 69.85 69.85) (xy 69.85 60.96))
     (stroke (width 0) (type default))
@@
     (stroke (width 0) (type default))
   )
+  (wire (pts (xy 95.25 110.49) (xy 116.84 110.49))
+    (stroke (width 0) (type default))
+  )
   (wire (pts (xy 66.04 82.55) (xy 69.85 82.55))
     (stroke (width 0) (type default))
@@
     (property "Intersheetrefs" "${INTERSHEET_REFS}" (at 108.1571 113.03 0)
       (effects (font (size 1.27 1.27)) (justify left) hide)
+    )
+  )
+  (symbol (lib_id "Device:D") (at 120.65 106.68 0) (unit 1)
+    (in_bom yes) (on_board yes) (dnp no)
+    (property "Reference" "D125" (at 120.65 104.14 0)
+      (effects (font (size 1.27 1.27)))
+    )
+    (property "Value" "SBA0530Q_R1_00001" (at 119.38 101.6 0)
+      (effects (font (size 1.27 1.27)))
+    )
+    (property "Footprint" "Diode_SMD:D_0402_1005Metric" (at 120.65 106.68 0)
+      (effects (font (size 1.27 1.27)) hide)
+    )
+    (property "Datasheet" "~" (at 120.65 106.68 0)
+      (effects (font (size 1.27 1.27)) hide)
+    )
+    (property "Sim.Device" "D" (at 120.65 106.68 0)
+      (effects (font (size 1.27 1.27)) hide)
+    )
+    (property "Sim.Pins" "1=K 2=A" (at 120.65 106.68 0)
+      (effects (font (size 1.27 1.27)) hide)
+    )
+    (pin "1")
+    (pin "2")
+    (instances
+      (project "gecko5education"
+        (path "/47d58937-9286-45a8-b88f-d3fcc6f916c8/1b790ed2-2ed7-44b0-8848-0151372cb9f5"
+          (reference "D125") (unit 1)
+        )
+        (path "/47d58937-9286-45a8-b88f-d3fcc6f916c8/2168b384-5196-4073-b8ef-3119545e18e5"
+          (reference "D123") (unit 1)
+        )
+      )
     )
   )
@@
         (path "/47d58937-9286-45a8-b88f-d3fcc6f916c8/1b790ed2-2ed7-44b0-8848-0151372cb9f5"
           (reference "D122") (unit 1)
-        )
-      )
-    )
-  )
-  (symbol (lib_id "power:+5V") (at 124.46 109.22 270) (unit 1)
-    (in_bom yes) (on_board yes) (dnp no) (fields_autoplaced)
-    (property "Reference" "#PWR090" (at 120.65 109.22 0)
-      (effects (font (size 1.27 1.27)) hide)
-    )
-    (property "Value" "+5V" (at 128.27 109.855 90)
-      (effects (font (size 1.27 1.27)) (justify left))
-    )
-    (property "Footprint" "" (at 124.46 109.22 0)
-      (effects (font (size 1.27 1.27)) hide)
-    )
-    (property "Datasheet" "" (at 124.46 109.22 0)
-      (effects (font (size 1.27 1.27)) hide)
-    )
-    (pin "1")
-    (instances
-      (project "gecko5education"
-        (path "/47d58937-9286-45a8-b88f-d3fcc6f916c8/1b790ed2-2ed7-44b0-8848-0151372cb9f5"
-          (reference "#PWR090") (unit 1)
         )
       )
@@
     )
   )
+  (symbol (lib_id "power:+5V") (at 125.73 107.95 270) (unit 1)
+    (in_bom yes) (on_board yes) (dnp no) (fields_autoplaced)
+    (property "Reference" "#PWR090" (at 121.92 107.95 0)
+      (effects (font (size 1.27 1.27)) hide)
+    )
+    (property "Value" "+5V" (at 129.54 108.585 90)
+      (effects (font (size 1.27 1.27)) (justify left))
+    )
+    (property "Footprint" "" (at 125.73 107.95 0)
+      (effects (font (size 1.27 1.27)) hide)
+    )
+    (property "Datasheet" "" (at 125.73 107.95 0)
+      (effects (font (size 1.27 1.27)) hide)
+    )
+    (pin "1")
+    (instances
+      (project "gecko5education"
+        (path "/47d58937-9286-45a8-b88f-d3fcc6f916c8/1b790ed2-2ed7-44b0-8848-0151372cb9f5"
+          (reference "#PWR090") (unit 1)
+        )
+      )
+    )
+  )
   (symbol (lib_id "power:GND") (at 97.79 134.62 0) (unit 1)
     (in_bom yes) (on_board yes) (dnp no) (fields_autoplaced)
@@
     )
   )
-  (symbol (lib_id "Device:D") (at 120.65 109.22 180) (unit 1)
-    (in_bom yes) (on_board yes) (dnp no) (fields_autoplaced)
-    (property "Reference" "D124" (at 120.65 102.87 0)
+  (symbol (lib_id "Device:D") (at 120.65 110.49 180) (unit 1)
+    (in_bom yes) (on_board yes) (dnp no)
+    (property "Reference" "D124" (at 120.65 113.03 0)
       (effects (font (size 1.27 1.27)))
     )
-    (property "Value" "SBA0530Q_R1_00001" (at 120.65 105.41 0)
+    (property "Value" "SBA0530Q_R1_00001" (at 121.92 115.57 0)
       (effects (font (size 1.27 1.27)))
     )
-    (property "Footprint" "Diode_SMD:D_0402_1005Metric" (at 120.65 109.22 0)
-      (effects (font (size 1.27 1.27)) hide)
-    )
-    (property "Datasheet" "~" (at 120.65 109.22 0)
-      (effects (font (size 1.27 1.27)) hide)
-    )
-    (property "Sim.Device" "D" (at 120.65 109.22 0)
-      (effects (font (size 1.27 1.27)) hide)
-    )
-    (property "Sim.Pins" "1=K 2=A" (at 120.65 109.22 0)
-      (effects (font (size 1.27 1.27)) hide)
-    )
+    (property "Footprint" "Diode_SMD:D_0402_1005Metric" (at 120.65 110.49 0)
+      (effects (font (size 1.27 1.27)) hide)
+    )
+    (property "Datasheet" "~" (at 120.65 110.49 0)
+      (effects (font (size 1.27 1.27)) hide)
+    )
+    (property "Sim.Device" "D" (at 120.65 110.49 0)
+      (effects (font (size 1.27 1.27)) hide)
+    )
+    (property "Sim.Pins" "1=K 2=A" (at 120.65 110.49 0)
+      (effects (font (size 1.27 1.27)) hide)
+    )
