File: kicad/GECKO5Education/sdram.kicad_sch (KiCad schematic)
At the start: 10 parts, among them U10 LP5907MFX-1.8, U11 MX25R3235FM2IL0, U6 LFE5U-85F-6BG381x, U9 IS42VM16160k-75BLI

Commit message: Final version
Parts:
- renumbered C15 to C17, C15 to C18, C15 to C19, R4 to R28, R4 to R29, R4 to R30
Changed lines of the file:
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@@
   (symbol (lib_id "Device:R") (at 82.55 137.16 0) (unit 1)
     (in_bom yes) (on_board yes) (dnp no)
-    (property "Reference" "R4" (at 81.28 130.81 90)
+    (property "Reference" "R29" (at 81.28 130.81 90)
       (effects (font (size 1.27 1.27)) (justify left))
     )
@@
     (instances
       (project "gecko5education"
-        (path "/47d58937-9286-45a8-b88f-d3fcc6f916c8"
-          (reference "R4") (unit 1)
-        )
-        (path "/47d58937-9286-45a8-b88f-d3fcc6f916c8/2168b384-5196-4073-b8ef-3119545e18e5"
-          (reference "R4") (unit 1)
-        )
         (path "/47d58937-9286-45a8-b88f-d3fcc6f916c8/0a7d71b4-2ae9-4114-b319-914176f8c7ac"
           (reference "R29") (unit 1)
@@
   (symbol (lib_id "Device:R") (at 80.01 137.16 0) (unit 1)
     (in_bom yes) (on_board yes) (dnp no)
-    (property "Reference" "R4" (at 78.74 130.81 90)
+    (property "Reference" "R28" (at 78.74 130.81 90)
       (effects (font (size 1.27 1.27)) (justify left))
     )
@@
     (instances
       (project "gecko5education"
-        (path "/47d58937-9286-45a8-b88f-d3fcc6f916c8"
-          (reference "R4") (unit 1)
-        )
-        (path "/47d58937-9286-45a8-b88f-d3fcc6f916c8/2168b384-5196-4073-b8ef-3119545e18e5"
-          (reference "R4") (unit 1)
-        )
         (path "/47d58937-9286-45a8-b88f-d3fcc6f916c8/0a7d71b4-2ae9-4114-b319-914176f8c7ac"
           (reference "R28") (unit 1)
@@
   (symbol (lib_id "Device:C") (at 76.2 33.02 0) (unit 1)
     (in_bom yes) (on_board yes) (dnp no) (fields_autoplaced)
-    (property "Reference" "C15" (at 80.01 32.385 0)
+    (property "Reference" "C18" (at 80.01 32.385 0)
       (effects (font (size 1.27 1.27)) (justify left))
     )
@@
     (instances
       (project "gecko5education"
-        (path "/47d58937-9286-45a8-b88f-d3fcc6f916c8/e8cfb843-efab-422d-aa9c-640a59ac0396"
-          (reference "C15") (unit 1)
-        )
         (path "/47d58937-9286-45a8-b88f-d3fcc6f916c8/0a7d71b4-2ae9-4114-b319-914176f8c7ac"
           (reference "C18") (unit 1)
@@
   (symbol (lib_id "Device:R") (at 77.47 137.16 0) (unit 1)
     (in_bom yes) (on_board yes) (dnp no)
-    (property "Reference" "R4" (at 76.2 130.81 90)
+    (property "Reference" "R30" (at 76.2 130.81 90)
       (effects (font (size 1.27 1.27)) (justify left))
     )
@@
     (instances
       (project "gecko5education"
-        (path "/47d58937-9286-45a8-b88f-d3fcc6f916c8"
-          (reference "R4") (unit 1)
-        )
-        (path "/47d58937-9286-45a8-b88f-d3fcc6f916c8/2168b384-5196-4073-b8ef-3119545e18e5"
-          (reference "R4") (unit 1)
-        )
         (path "/47d58937-9286-45a8-b88f-d3fcc6f916c8/0a7d71b4-2ae9-4114-b319-914176f8c7ac"
           (reference "R30") (unit 1)
@@
   (symbol (lib_id "Device:C") (at 88.9 33.02 0) (unit 1)
     (in_bom yes) (on_board yes) (dnp no) (fields_autoplaced)
-    (property "Reference" "C15" (at 92.71 32.385 0)
+    (property "Reference" "C19" (at 92.71 32.385 0)
       (effects (font (size 1.27 1.27)) (justify left))
     )
@@
     (instances
       (project "gecko5education"
-        (path "/47d58937-9286-45a8-b88f-d3fcc6f916c8/e8cfb843-efab-422d-aa9c-640a59ac0396"
-          (reference "C15") (unit 1)
-        )
         (path "/47d58937-9286-45a8-b88f-d3fcc6f916c8/0a7d71b4-2ae9-4114-b319-914176f8c7ac"
           (reference "C19") (unit 1)
@@
   (symbol (lib_id "Device:C") (at 49.53 33.02 0) (unit 1)
     (in_bom yes) (on_board yes) (dnp no) (fields_autoplaced)
-    (property "Reference" "C15" (at 53.34 32.385 0)
+    (property "Reference" "C17" (at 53.34 32.385 0)
       (effects (font (size 1.27 1.27)) (justify left))
     )
@@
     (instances
       (project "gecko5education"
-        (path "/47d58937-9286-45a8-b88f-d3fcc6f916c8/e8cfb843-efab-422d-aa9c-640a59ac0396"
-          (reference "C15") (unit 1)
-        )
         (path "/47d58937-9286-45a8-b88f-d3fcc6f916c8/0a7d71b4-2ae9-4114-b319-914176f8c7ac"
           (reference "C17") (unit 1)
