File: kicad/GECKO5Education/switches.kicad_sch (KiCad schematic)
At the start: 31 parts, among them Q1 BC807, Q2 BC807, Q3 BC807, Q4 BC807, Q5 BC807, SW1 SW_Push, SW2 SW_Push, SW3 SW_Push, SW4 SW_Push, SW5 SW_Push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

Commit message: Final version
Parts:
- renumbered C15 to C21, R1 to R32, R1 to R33, R1 to R34, R1 to R35, R1 to R36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
