File: kicad/GECKO5Education/usbHub.kicad_sch (KiCad schematic)
At the start: 24 parts, among them SW7 B3U-1000P[], U15 SN74HC266DR, U19 USB2513B-AEZC

Commit message: Changed the USB-reset to reset the FPGA to reconfigure instead of applying the "reset" button, which makes more sense in a system reset
Connections:
- net nResetFPGA renamed nProgramFpga
Changed lines of the file:
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@@
     )
   )
-  (global_label "nResetFPGA" (shape output) (at 151.13 156.21 0) (fields_autoplaced)
+  (global_label "nProgramFpga" (shape output) (at 151.13 156.21 0) (fields_autoplaced)
     (effects (font (size 1.27 1.27)) (justify left))
-    (property "Intersheetrefs" "${INTERSHEET_REFS}" (at 165.1824 156.21 0)
+    (property "Intersheetrefs" "${INTERSHEET_REFS}" (at 167.7825 156.21 0)
       (effects (font (size 1.27 1.27)) (justify left) hide)
     )
