File: kicad/GECKO5Education/led_array.kicad_sch (KiCad schematic)
At the start: 181 parts, among them Q10 BC807, Q11 BC807, Q12 BC807, Q13 BC807, Q14 BC807, Q15 BC807, Q16 BC807, Q17 BC807, Q6 BC807, Q7 BC807, Q8 BC807, Q9 BC807, U5 74HC154BQ,118, U6 LFE5U-85F-6BG381x

Commit message: Production version EPFL
Parts:
- D10, D100, D101, D102, D103, D104, D105, D106, D107, D108, D109, D11, D110, D111, D112, D113, D114, D115, D116, D117, D118, D119, D12, D120, D121, D13, D14, D15, D16, D17, D18, D19, D2, D20, D21, D22, D23, D24, D25, D26, D27, D28, D29, D3, D30, D31, D32, D33, D34, D35, D36, D37, D38, D39, D4, D40, D41, D42, D43, D44, D45, D46, D47, D48, D49, D5, D50, D51, D52, D53, D54, D55, D56, D57, D58, D59, D6, D60, D61, D62, D63, D64, D65, D66, D67, D68, D69, D7, D70, D71, D72, D73, D74, D75, D76, D77, D78, D79, D8, D80, D81, D82, D83, D84, D85, D86, D87, D88, D89, D9, D90, D91, D92, D93, D94, D95, D96, D97, D98, D99: symbol Device:LED_ARGB -> gecko5education:EAST1616RGBB2
Connections:
- net at D74.2 (GK), D75.2 (GK), D76.2 (GK)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: now also R83.2; no longer R82.2
- net at D74.3 (BK), D75.3 (BK), D76.3 (BK)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: now also R84.2; no longer R83.2
- net at D14.2 (GK), D15.2 (GK), D16.2 (GK)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: now also R68.2; no longer R67.2
- net at D14.3 (BK), D15.3 (BK), D16.3 (BK)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: now also R69.2; no longer R68.2
- net at D86.3 (BK), D87.3 (BK), D88.3 (BK)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: now also R87.2; no longer R86.2
- net at D62.2 (GK), D63.2 (GK), D64.2 (GK)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: now also R80.2; no longer R79.2
- net at D62.3 (BK), D63.3 (BK), D64.3 (BK)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: now also R81.2; no longer R80.2
- net at D26.2 (GK), D27.2 (GK), D28.2 (GK)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: now also R71.2; no longer R70.2
- net at D10.2 (GK), D11.2 (GK), D12.2 (GK)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: now also R65.2; no longer R64.2
- net at D10.3 (BK), D11.3 (BK), D12.3 (BK)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: now also R66.2; no longer R65.2
- net at D50.3 (BK), D51.3 (BK), D52.3 (BK)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: now also R78.2; no longer R77.2
- net at D38.2 (GK), D39.2 (GK), D40.2 (GK)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: now also R74.2; no longer R73.2
- net at D38.3 (BK), D39.3 (BK), D40.3 (BK)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: now also R75.2; no longer R74.2
- net at D26.3 (BK), D27.3 (BK), D28.3 (BK)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: now also R72.2; no longer R71.2
- net at D100.2 (GK), D101.2 (GK), D102.2 (GK)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: now also R89.2; no longer R88.2
- net at D100.3 (BK), D101.3 (BK), D102.3 (BK)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: now also R90.2; no longer R89.2
- net at D110.2 (GK), D111.2 (GK), D112.2 (GK)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: now also R92.2; no longer R91.2
- net at D110.3 (BK), D111.3 (BK), D112.3 (BK)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: now also R93.2; no longer R92.2
- net at D50.2 (GK), D51.2 (GK), D52.2 (GK)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: now also R77.2; no longer R76.2
- net at D86.2 (GK), D87.2 (GK), D88.2 (GK)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: now also R86.2; no longer R85.2
- new net: D74.1 (RK), D75.1 (RK), D76.1 (RK), D77.1 (RK), D78.1 (RK), D79.1 (RK), D80.1 (RK), D81.1 (RK), D82.1 (RK), D83.1 (RK), D84.1 (RK), D85.1 (RK), R82.2
- new net: D107.4 (A), D11.4 (A), D119.4 (A), D23.4 (A), D35.4 (A), D47.4 (A), D59.4 (A), D71.4 (A), D83.4 (A), D95.4 (A), Q15.3 (C)
- new net: D14.1 (RK), D15.1 (RK), D16.1 (RK), D17.1 (RK), D18.1 (RK), D19.1 (RK), D20.1 (RK), D21.1 (RK), D22.1 (RK), D23.1 (RK), D24.1 (RK), D25.1 (RK), R67.2
- new net: D108.4 (A), D12.4 (A), D120.4 (A), D24.4 (A), D36.4 (A), D48.4 (A), D60.4 (A), D72.4 (A), D84.4 (A), D96.4 (A), Q16.3 (C)
- new net: D62.1 (RK), D63.1 (RK), D64.1 (RK), D65.1 (RK), D66.1 (RK), D67.1 (RK), D68.1 (RK), D69.1 (RK), D70.1 (RK), D71.1 (RK), D72.1 (RK), D73.1 (RK), R79.2
- new net: D100.4 (A), D112.4 (A), D16.4 (A), D28.4 (A), D4.4 (A), D40.4 (A), D52.4 (A), D64.4 (A), D76.4 (A), D88.4 (A), Q8.3 (C)
- new net: D26.1 (RK), D27.1 (RK), D28.1 (RK), D29.1 (RK), D30.1 (RK), D31.1 (RK), D32.1 (RK), D33.1 (RK), D34.1 (RK), D35.1 (RK), D36.1 (RK), D37.1 (RK), R70.2
- new net: D10.1 (RK), D11.1 (RK), D12.1 (RK), D13.1 (RK), D2.1 (RK), D3.1 (RK), D4.1 (RK), D5.1 (RK), D6.1 (RK), D7.1 (RK), D8.1 (RK), D9.1 (RK), R64.2
- new net: D102.4 (A), D114.4 (A), D18.4 (A), D30.4 (A), D42.4 (A), D54.4 (A), D6.4 (A), D66.4 (A), D78.4 (A), D90.4 (A), Q10.3 (C)
- new net: D38.1 (RK), D39.1 (RK), D40.1 (RK), D41.1 (RK), D42.1 (RK), D43.1 (RK), D44.1 (RK), D45.1 (RK), D46.1 (RK), D47.1 (RK), D48.1 (RK), D49.1 (RK), R73.2
- new net: D110.4 (A), D14.4 (A), D2.4 (A), D26.4 (A), D38.4 (A), D50.4 (A), D62.4 (A), D74.4 (A), D86.4 (A), D98.4 (A), Q6.3 (C)
- new net: D104.4 (A), D116.4 (A), D20.4 (A), D32.4 (A), D44.4 (A), D56.4 (A), D68.4 (A), D8.4 (A), D80.4 (A), D92.4 (A), Q12.3 (C)
- new net: D103.4 (A), D115.4 (A), D19.4 (A), D31.4 (A), D43.4 (A), D55.4 (A), D67.4 (A), D7.4 (A), D79.4 (A), D91.4 (A), Q11.3 (C)
- new net: D105.4 (A), D117.4 (A), D21.4 (A), D33.4 (A), D45.4 (A), D57.4 (A), D69.4 (A), D81.4 (A), D9.4 (A), D93.4 (A), Q13.3 (C)
- new net: D101.4 (A), D113.4 (A), D17.4 (A), D29.4 (A), D41.4 (A), D5.4 (A), D53.4 (A), D65.4 (A), D77.4 (A), D89.4 (A), Q9.3 (C)
- new net: D100.1 (RK), D101.1 (RK), D102.1 (RK), D103.1 (RK), D104.1 (RK), D105.1 (RK), D106.1 (RK), D107.1 (RK), D108.1 (RK), D109.1 (RK), D98.1 (RK), D99.1 (RK), R88.2
- new net: D10.4 (A), D106.4 (A), D118.4 (A), D22.4 (A), D34.4 (A), D46.4 (A), D58.4 (A), D70.4 (A), D82.4 (A), D94.4 (A), Q14.3 (C)
- new net: D110.1 (RK), D111.1 (RK), D112.1 (RK), D113.1 (RK), D114.1 (RK), D115.1 (RK), D116.1 (RK), D117.1 (RK), D118.1 (RK), D119.1 (RK), D120.1 (RK), D121.1 (RK), R91.2
- new net: D50.1 (RK), D51.1 (RK), D52.1 (RK), D53.1 (RK), D54.1 (RK), D55.1 (RK), D56.1 (RK), D57.1 (RK), D58.1 (RK), D59.1 (RK), D60.1 (RK), D61.1 (RK), R76.2
- new net: D109.4 (A), D121.4 (A), D13.4 (A), D25.4 (A), D37.4 (A), D49.4 (A), D61.4 (A), D73.4 (A), D85.4 (A), D97.4 (A), Q17.3 (C)
- new net: D111.4 (A), D15.4 (A), D27.4 (A), D3.4 (A), D39.4 (A), D51.4 (A), D63.4 (A), D75.4 (A), D87.4 (A), D99.4 (A), Q7.3 (C)
- new net: D86.1 (RK), D87.1 (RK), D88.1 (RK), D89.1 (RK), D90.1 (RK), D91.1 (RK), D92.1 (RK), D93.1 (RK), D94.1 (RK), D95.1 (RK), D96.1 (RK), D97.1 (RK), R85.2

Commit message: Cleaned up
Parts:
- D10, D100, D101, D102, D103, D104, D105, D106, D107, D108, D109, D11, D110, D111, D112, D113, D114, D115, D116, D117, D118, D119, D12, D120, D121, D13, D14, D15, D16, D17, D18, D19, D2, D20, D21, D22, D23, D24, D25, D26, D27, D28, D29, D3, D30, D31, D32, D33, D34, D35, D36, D37, D38, D39, D4, D40, D41, D42, D43, D44, D45, D46, D47, D48, D49, D5, D50, D51, D52, D53, D54, D55, D56, D57, D58, D59, D6, D60, D61, D62, D63, D64, D65, D66, D67, D68, D69, D7, D70, D71, D72, D73, D74, D75, D76, D77, D78, D79, D8, D80, D81, D82, D83, D84, D85, D86, D87, D88, D89, D9, D90, D91, D92, D93, D94, D95, D96, D97, D98, D99: value XZCMEDGCBD110W -> EAST1616RGBB2; footprint gecko4education:RGB_LED -> gecko4education:EAST1616RGBB2_EVE
