File: kicad/perifAddOn/perifAddOn.kicad_pcb (KiCad board)
At the start: 4 copper layers, 60.6 x 75.2 mm, 70 parts, among them J1 QTE-020-01-X-D-A, J2 105450-0101, J3 GTFP08431BEU, J4 Conn_02x15_Odd_Even, J5 Conn_02x15_Odd_Even, SW1 B3U-1000P[], SW2 B3U-1000P[], SW3 B3U-1000P[], U1 AP2281-3WG-7, U2 SN74HC266DR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

Commit message: Added bom
Other:
- board text added: "Version 1.0"
Changed lines of the file:
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@@
+    (effects (font (size 1 1) (thickness 0.15)) (justify left bottom))
+  )
+  (gr_text "Version 1.0\n" (at 108.9 91.45) (layer "F.SilkS")
     (effects (font (size 1 1) (thickness 0.15)) (justify left bottom))
   )

Commit message: lates version
Connections:
- J4 pad 24: GND -> unconnected-(J4-Pin_24-Pad24)
Changed lines of the file:
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@@
   (net 129 "unconnected-(J4-Pin_17-Pad17)")
   (net 130 "unconnected-(J4-Pin_18-Pad18)")
+  (net 131 "unconnected-(J4-Pin_24-Pad24)")
   (footprint "Resistor_SMD:R_0402_1005Metric" (layer "F.Cu")
     (at 99.4 46.4 180)
@@
     (pad "23" thru_hole oval (at 0 27.94 270) (size 1.7 1.7) (drill 1) (layers "*.Cu" "*.Mask") (remove_unused_layers) (keep_end_layers) (zone_layer_connections)
       (net 124 "VREF") (pinfunction "Pin_23") (pintype "passive"))
-    (pad "24" thru_hole oval (at 2.54 27.94 270) (size 1.7 1.7) (drill 1) (layers "*.Cu" "*.Mask") (remove_unused_layers) (keep_end_layers) (zone_layer_connections "In1.Cu")
-      (net 6 "GND") (pinfunction "Pin_24") (pintype "passive"))
+    (pad "24" thru_hole oval (at 2.54 27.94 270) (size 1.7 1.7) (drill 1) (layers "*.Cu" "*.Mask") (remove_unused_layers) (keep_end_layers) (zone_layer_connections)
+      (net 131 "unconnected-(J4-Pin_24-Pad24)") (pinfunction "Pin_24") (pintype "passive+no_connect"))
     (pad "25" thru_hole oval (at 0 30.48 270) (size 1.7 1.7) (drill 1) (layers "*.Cu" "*.Mask") (remove_unused_layers) (keep_end_layers) (zone_layer_connections "In1.Cu")
       (net 6 "GND") (pinfunction "Pin_25") (pintype "passive"))
