File: kicad/perifAddOn/perifAddOn.kicad_pcb (KiCad board)
At the start: 4 copper layers, 60.6 x 75.2 mm, 70 parts, among them J1 QTE-020-01-X-D-A, J2 105450-0101, J3 GTFP08431BEU, J4 Conn_02x15_Odd_Even, J5 Conn_02x15_Odd_Even, SW1 B3U-1000P[], SW2 B3U-1000P[], SW3 B3U-1000P[], U1 AP2281-3WG-7, U2 SN74HC266DR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

Commit message: V1.1 of perifAddOn (added bus-switch on sd-card)
Parts:
- added U7: TC7MBL3245CFTEL, addOnTemplate:TSSOP20_TOS, F.Cu at (97.2, 64.5)
- moved C18 5.66 mm to (131.9, 48.2)
- moved R18 5.66 mm to (143.9, 58.2)
- moved C15 5.66 mm to (133.2, 48.4)
- moved C19 5.66 mm to (130.2, 53.3)
- moved R17 5.66 mm to (133.2, 50.2)
- moved SW2 5.66 mm to (132.2, 54.5)
- moved SW3 5.66 mm to (146.9, 58.9)
- moved U5 5.66 mm to (140.8, 48.6)
- moved Y1 5.66 mm to (136.2, 58.2)
- moved C16 4.16 mm to (138.5, 58.2), turned to 0 degrees
- moved C17 3.97 mm to (134.0, 58.2), turned to 180 degrees
Connections:
- J1 pad 03: SdD0 -> SdD0B
- J1 pad 04: SdnDet -> SdnDetB
- J1 pad 05: SdD1 -> SdD1B
- J1 pad 06: SdD2 -> SdD2B
- J1 pad 08: SdD3 -> SdD3B
- J1 pad 10: SdCmd -> SdCmdB
- J1 pad 12: SdClk -> SdClkB
- R10 pad 1: +3.3V -> GND
Routing:
- net SDCnReset: track 31.2 -> 47.6 mm, vias 2 -> 3
- net SdClkB: track 0.00 -> 11.2 mm, vias 0 -> 1
- net SdCmdB: track 0.00 -> 10.4 mm, vias 0 -> 1
- net EspIO3: track 38.9 -> 29.4 mm
- net SdD3B: track 0.00 -> 9.18 mm, vias 0 -> 1
- net SdD1B: track 0.00 -> 8.96 mm, vias 0 -> 1
- net SdD2B: track 0.00 -> 8.38 mm, vias 0 -> 1
- net GND: track 86.5 -> 94.8 mm, vias 61 -> 62
- net SdD1: track 41.8 -> 50.0 mm, vias 1 -> 0
- net SdD0B: track 0.00 -> 8.12 mm, vias 0 -> 1
- net SdnDetB: track 0.00 -> 7.45 mm, vias 0 -> 1
- net SdD3: track 46.7 -> 40.2 mm, vias 1 -> 0
- net SdD2: track 46.9 -> 41.5 mm, vias 1 -> 0
- net EspEnable: track 28.7 -> 24.8 mm
- net SdnDet: track 57.3 -> 53.5 mm, vias 3 -> 2
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Other:
- outline, holes or cut-outs redrawn
- board text added: "TJHK 2024"
- board text added: "Version 1.1"
- board text removed: "TJHK 2023"
- board text removed: "Version 1.0"
