File: kicad/perifAddOn/pmod.kicad_sch (KiCad schematic)
At the start: 2 parts, among them J4 Conn_02x15_Odd_Even, J5 Conn_02x15_Odd_Even

Commit message: lates version
Connections:
- net GND: no longer J4.24 (Pin_24)
- no-connect marks 2 -> 3
Changed lines of the file:
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@@
   (junction (at 46.99 64.77) (diameter 0) (color 0 0 0 0)
-  )
-  (junction (at 46.99 57.15) (diameter 0) (color 0 0 0 0)
   )
   (junction (at 102.87 45.72) (diameter 0) (color 0 0 0 0)
   )
+  (no_connect (at 45.72 57.15))
   (no_connect (at 33.02 49.53))
   (no_connect (at 45.72 49.53))
@@
   )
   (wire (pts (xy 30.48 34.29) (xy 33.02 34.29))
-    (stroke (width 0) (type default))
-  )
-  (wire (pts (xy 46.99 57.15) (xy 46.99 59.69))
     (stroke (width 0) (type default))
   )
@@
     (stroke (width 0) (type default))
   )
-  (wire (pts (xy 45.72 57.15) (xy 46.99 57.15))
-    (stroke (width 0) (type default))
-  )
   (wire (pts (xy 86.36 55.88) (xy 88.9 55.88))
     (stroke (width 0) (type default))
@@
     (stroke (width 0) (type default))
   )
-  (wire (pts (xy 46.99 52.07) (xy 46.99 57.15))
+  (wire (pts (xy 46.99 52.07) (xy 46.99 59.69))
     (stroke (width 0) (type default))
   )
