File: kicad/lcdAddOn/mseAddOn.kicad_pcb (KiCad board)
At the start: 2 copper layers, 60.6 x 100 mm, 14 parts, among them J1 QTE-020-01-F-D-A, J2 62684-402100ALF, U1 AR1021-I/SS

Commit message: latest version with camera
Parts:
- added SW1: SW_Push, addOnTemplate:pushbutton, F.Cu at (103.2, 135.4)
- added SW2: SW_Push, addOnTemplate:pushbutton, F.Cu at (117.1, 135.5)
- added SW3: SW_Push, addOnTemplate:pushbutton, F.Cu at (131.1, 135.6)
- moved J2 43.1 mm to (94.3, 64.2), turned to 90 degrees
- moved R4 37.2 mm to (95.5, 78.8)
- moved R3 36.4 mm to (96.5, 78.8)
- moved R2 35.6 mm to (97.4, 78.8)
- moved R1 34.9 mm to (98.4, 78.8)
- moved C1 34.2 mm to (102.9, 84.5)
- moved C2 34.2 mm to (102.8, 86.5)
- moved C3 34.2 mm to (91.0, 83.8)
- moved U1 34.2 mm to (96.9, 86.8)
- moved R5 34.2 mm to (98.7, 82.0)
Connections:
- J1 pad 03: IMO -> DB11
- J1 pad 04: unconnected-(J1-Pad04) -> Net-(J1-Pad04)
- J1 pad 05: FMARK -> DB10
- J1 pad 06: unconnected-(J1-Pad06) -> Net-(J1-Pad06)
- J1 pad 07: RESET -> DB9
- J1 pad 08: unconnected-(J1-Pad08) -> Net-(J1-Pad08)
- J1 pad 09: RS -> DB8
- J1 pad 10: SDO -> DB12
- J1 pad 11: CS -> DB7
- J1 pad 12: SS -> DB13
- J1 pad 13: RD -> DB6
- J1 pad 14: SIQ -> DB14
- J1 pad 15: WR -> DB0
- J1 pad 16: M1 -> DB15
- J1 pad 17: DB15 -> DB1
- J1 pad 18: SCK/SCL -> WR
- J1 pad 19: DB14 -> DB2
- J1 pad 20: SDI/SDA -> RD
- J1 pad 21: DB13 -> DB3
- J1 pad 22: DB5 -> CS
- J1 pad 23: DB12 -> DB4
- J1 pad 24: DB4 -> RS
- J1 pad 25: DB11 -> DB5
- J1 pad 26: DB3 -> RESET
- J1 pad 27: DB10 -> SDI/SDA
- J1 pad 28: DB2 -> FMARK
- J1 pad 29: DB9 -> SCK/SCL
- J1 pad 30: DB1 -> IMO
- J1 pad 31: DB8 -> M1
- J1 pad 33: DB7 -> SIQ
- J1 pad 35: DB6 -> SS
- J1 pad 37: DB0 -> SDO
- J2 pad 41: GND -> (no net)
- J2 pad 42: GND -> (no net)
Routing:
- net Net-(J1-Pad04): track 0.00 -> 151.2 mm, vias 0 -> 1
- net Net-(J1-Pad06): track 0.00 -> 133.4 mm, vias 0 -> 1
- net Net-(J1-Pad08): track 0.00 -> 117.3 mm, vias 0 -> 1
- net SCK/SCL: track 119.3 -> 31.4 mm
- net SDO: track 138.2 -> 52.0 mm
- net SDI/SDA: track 116.1 -> 30.1 mm
- net SS: track 135.9 -> 54.7 mm
- net SIQ: track 133.6 -> 57.8 mm
- net M1: track 133.3 -> 62.9 mm
- net DB5: track 75.0 -> 30.2 mm
- net DB4: track 73.2 -> 29.3 mm
- net DB3: track 71.6 -> 28.3 mm
- net DB2: track 69.7 -> 27.4 mm
- net DB1: track 67.6 -> 26.4 mm
- net DB11: track 47.2 -> 18.7 mm
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Other:
- board text added: "GECKO5Education LCD-add-on"
- board text added: "PB1"
- board text added: "PB2"
- board text added: "PB3"
- board text added: "TJHK2024"
- board text added: "Version 1.0"
