File: kicad/lcdAddOn/mseAddOn.kicad_sch (KiCad schematic)
At the start: 11 parts, among them J1 QTE-020-01-F-D-A, J2 62684-402100ALF, U1 AR1021-I/SS

Commit message: latest version with camera
Parts:
- added SW1, SW2, SW3: SW_Push, addOnTemplate:pushbutton, symbol Switch:SW_Push
Connections:
- net CS: now also J1.22; no longer J1.11
- net DB0: now also J1.15; no longer J1.37
- net DB1: now also J1.17; no longer J1.30
- net DB10: now also J1.05; no longer J1.27
- net DB11: now also J1.03; no longer J1.25
- net DB12: now also J1.10; no longer J1.23
- net DB13: now also J1.12; no longer J1.21
- net DB14: now also J1.14; no longer J1.19
- net DB15: now also J1.16; no longer J1.17
- net DB2: now also J1.19; no longer J1.28
- net DB3: now also J1.21; no longer J1.26
- net DB4: now also J1.23; no longer J1.24
- net DB5: now also J1.25; no longer J1.22
- net DB6: now also J1.13; no longer J1.35
- net DB7: now also J1.11; no longer J1.33
- net DB8: now also J1.09; no longer J1.31
- net DB9: now also J1.07; no longer J1.29
- net FMARK: now also J1.28; no longer J1.05
- net GND: now also SW1.2, SW2.2, SW3.2
- net IMO: now also J1.30; no longer J1.03
- net M1: now also J1.31; no longer J1.16
- net RD: now also J1.20; no longer J1.13
- net RESET: now also J1.26; no longer J1.07
- net RS: now also J1.24; no longer J1.09
- net SCK/SCL: now also J1.29; no longer J1.18
- net SDI/SDA: now also J1.27; no longer J1.20
- net SDO: now also J1.37; no longer J1.10
- net SIQ: now also J1.33; no longer J1.14
- net SS: now also J1.35; no longer J1.12
- net WR: now also J1.18; no longer J1.15
- net at J1.04: now also SW1.1
- net at J1.06: now also SW2.1
- net at J1.08: now also SW3.1
- no-connect marks 11 -> 6
Other:
- moved on the sheet: J2, R1, R2, R3, R4
